Commit message: refactor simpleHumanoid -> simple-humanoid

File: data/urdf/simple_humanoid_lleg_rom.urdf (robot description, URDF)
Before this commit: robot simpleHumanoid_rleg_rom, 1 links, 0 joints
Links:
- removed link rleg_rom
- added link llged_rom; collision mesh filename=package://simple-humanoid-rbprm/meshes/Lleg_rom.stl; visual mesh filename=package://simple-humanoid-rbprm/meshes/Lleg_rom.stl

File: data/urdf/simple_humanoid_rleg_rom.urdf (robot description, URDF)
Before this commit: robot simpleHumanoid_lleg_rom, 1 links, 0 joints
Links:
- removed link llged_rom
- added link rleg_rom; collision mesh filename=package://simple-humanoid-rbprm/meshes/Rleg_rom.stl; visual mesh filename=package://simple-humanoid-rbprm/meshes/Rleg_rom.stl
